Commit message: Model head camera as RealSense D455

File: configs/assembly.urdf (robot description, URDF)
Before this commit: robot tron2_dach_revo3_supplied_step_brackets, 107 links, 106 joints
Links:
- link head_camera_link: geometry visual box size=0.026 0.124 0.029
Joints:
- joint head_camera_color_joint: origin xyz=0 0.015 0 rpy=0 0 0 -> xyz=0 -0.059 0 rpy=0 0 0
- joint head_camera_link_joint: origin xyz=0.0106 0.0175 0.0125 rpy=0 0 0 -> xyz=0.01115 0.0475 0.0145 rpy=0 0 0
